Commit message: Fixed geometry issues with constraints on box pushing

File: spline_rl/urdf/panda.urdf (robot description, URDF)
Before this commit: robot panda, 12 links, 11 joints
Links:
- added link panda_push_rod; collision cylinder length=0.15 radius=0.01; visual cylinder length=0.15 radius=0.01
- added link push_rod_tip; collision box size=0.01 0.01 0.01; visual box size=0.01 0.01 0.01
Joints:
- added joint panda_push_rod_joint: type fixed, parent panda_hand, child panda_push_rod, origin xyz=0 0 0 rpy=0 0 0
- added joint push_rod_tip_joint: type fixed, parent panda_push_rod, child push_rod_tip, origin xyz=0 0 0.20 rpy=0 0 0
